File: Hall effect endstop/PCK-HALL.kicad_sch (KiCad schematic)
At the start: 7 parts, among them IC1 TMAG5328A1ZQDBVR, J1 Conn_01x03

Commit message: As built update
Parts:
- R1: value TBD -> 11k
Changed lines of the file:
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@@
 			)
 		)
-		(property "Value" "TBD"
+		(property "Value" "11k"
 			(at 119.634 115.57 0)
 			(effects
