File: Camera connector/Camera_connector_board/Camera_connector_board.kicad_pcb (KiCad board)
At the start: 2 copper layers, 15.2 x 29 mm, 4 parts, among them J1 SJ-2524-SMT-TR, J2 Conn_01x03

Commit message: V1.0 - manufacturing
Other:
- board text added: "Camera breakout board v1.0"
- board text added: "PCK-ST1"
