File: Main board/MCU.kicad_sch (KiCad schematic)
At the start: 53 parts, among them J1 RPi, J10 RA, J11 EL, J12 AZ, J13 GPS, J14 SHUTTER, J15 PWR_ON, J2 RJE05-166-1310, J9 DEC, Q1 2N7002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

Commit message: sch update
Changed lines of the file:
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@@
 					(size 1.27 1.27)
 				)
+				(hide yes)
 			)
 		)
@@
 					(size 1.27 1.27)
 				)
-			)
-		)
+				(hide yes)
+			)
+		)
