File: Main board/PCK-ST1.kicad_sch (KiCad schematic)
At the start: 21 parts

Commit message: sch update
Other:
- moved on the sheet: C54, C55, R18, R19, R20, R21, R22, R23, R24, R25, R28, R29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
