File: Main board/Power_delivery.kicad_sch (KiCad schematic)
At the start: 25 parts, among them IC8 TPS25730DREFR, J7 USB_C_Receptacle_USB2.0_16P

Commit message: Main board updated to v0.3
Parts:
- TP5: footprint TestPoint:TestPoint_Pad_D1.5mm -> TestPoint:TestPoint_Pad_D1.0mm
Changed lines of the file:
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@@
 			)
 		)
-		(property "Footprint" "TestPoint:TestPoint_Pad_D1.5mm"
+		(property "Footprint" "TestPoint:TestPoint_Pad_D1.0mm"
 			(at 154.94 34.29 0)
 			(effects

Commit message: Main board v0.3 to be manufactured
Other:
- moved on the sheet: R64
Changed lines of the file:
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@@
 	(wire
 		(pts
-			(xy 191.77 123.19) (xy 199.39 123.19)
+			(xy 191.77 123.19) (xy 210.82 123.19)
 		)
 		(stroke
@@
 	(wire
 		(pts
+			(xy 210.82 114.3) (xy 210.82 110.49)
+		)
+		(stroke
+			(width 0)
+			(type default)
+		)
+	)
+	(wire
+		(pts
 			(xy 148.59 125.73) (xy 147.32 125.73)
 		)
@@
 	(wire
 		(pts
-			(xy 210.82 123.19) (xy 210.82 110.49)
+			(xy 210.82 123.19) (xy 210.82 121.92)
 		)
 		(stroke
@@
 	(wire
 		(pts
-			(xy 210.82 123.19) (xy 207.01 123.19)
-		)
-		(stroke
-			(width 0)
-			(type default)
-		)
-	)
-	(wire
-		(pts
 			(xy 78.74 118.11) (xy 74.93 118.11)
 		)
@@
 	(symbol
 		(lib_id "Device:R")
-		(at 203.2 123.19 270)
+		(at 210.82 118.11 0)
 		(unit 1)
 		(exclude_from_sim no)
@@
 		(dnp no)
 		(property "Reference" "R64"
-			(at 203.1072 119.38 90)
+			(at 207.518 117.094 0)
 			(effects
 				(font
@@
 		)
 		(property "Value" "100k"
-			(at 203.1072 121.158 90)
+			(at 207.264 119.126 0)
 			(effects
 				(font
@@
 		)
 		(property "Footprint" "Resistor_SMD:R_0402_1005Metric"
-			(at 203.2 121.412 90)
+			(at 209.042 118.11 90)
 			(effects
 				(font
@@
 		)
 		(property "Datasheet" "~"
-			(at 203.2 123.19 0)
+			(at 210.82 118.11 0)
 			(effects
 				(font
@@
 		)
 		(property "Description" "Resistor"
-			(at 203.2 123.19 0)
+			(at 210.82 118.11 0)
 			(effects
 				(font

Commit message: Added part numbers for simpler ordering
Parts:
- C10, C9: Part Number (none) -> GRM1555C2A391JE01D
- C11: Part Number (none) -> C3216X5R1E476M160AC
- C4, C6, C7: Part Number (none) -> GRM155R61A106ME11D
- C8: Part Number (none) -> GRM188R61E475KE11D
- D1: Part Number (none) -> TPD4E05U06DQAR
- D2: Part Number (none) -> SMF22A-E3-08
- IC8: Part Number (none) -> TPS25730DREFR
- J7, TP5: now left out of the parts list
- R45, R46, R47, R48, R49, R64: Part Number (none) -> CRCW0402100KFKEE
- R6, R8: Alternative PN (none) -> RCC0402200KFKED; Part Number (none) -> CRCW0402200KFKEDHP
- R61: Part Number (none) -> CRCW0402200KFKEDHP
- R62, R7: Part Number (none) -> CRCW040224K0FKEDC
- R63: Part Number (none) -> CRCW04020000Z0EDC
- R9: Part Number (none) -> CRCW040210K0FKEDC
Changed lines of the file:
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@@
+			)
+		)
+		(property "Part Number" "SMF22A-E3-08"
+			(at 104.14 125.73 0)
+			(effects
+				(font
+					(size 1.27 1.27)
+				)
+				(hide yes)
 			)
 		)
@@
 			)
 		)
+		(property "Part Number" "GRM1555C2A391JE01D"
+			(at 121.666 101.346 0)
+			(effects
+				(font
+					(size 1.27 1.27)
+				)
+				(hide yes)
+			)
+		)
 		(pin "2"
 		)
@@
 			)
 		)
+		(property "Part Number" "GRM155R61A106ME11D"
+			(at 120.65 44.45 0)
+			(effects
+				(font
+					(size 1.27 1.27)
+				)
+				(hide yes)
+			)
+		)
 		(pin "2"
 		)
@@
 			)
 		)
+		(property "Part Number" "CRCW040224K0FKEDC"
+			(at 243.84 113.03 0)
+			(effects
+				(font
+					(size 1.27 1.27)
+				)
+				(hide yes)
+			)
+		)
 		(pin "2"
 		)
@@
 		)
 		(property "Description" "Resistor"
+			(at 203.2 110.49 0)
+			(effects
+				(font
+					(size 1.27 1.27)
+				)
+				(hide yes)
+			)
+		)
+		(property "Part Number" "CRCW0402100KFKEE"
 			(at 203.2 110.49 0)
 			(effects
@@
 			)
 		)
+		(property "Part Number" "CRCW0402200KFKEDHP"
+			(at 251.46 97.79 0)
+			(effects
+				(font
+					(size 1.27 1.27)
+				)
+				(hide yes)
+			)
+		)
 		(pin "2"
 		)
@@
 		(unit 1)
 		(exclude_from_sim no)
-		(in_bom yes)
+		(in_bom no)
 		(on_board yes)
 		(dnp no)
@@
 			)
 		)
+		(property "Part Number" "CRCW040224K0FKEDC"
+			(at 251.46 113.03 0)
+			(effects
+				(font
+					(size 1.27 1.27)
+				)
+				(hide yes)
+			)
+		)
 		(pin "2"
 		)
@@
 			)
 		)
+		(property "Part Number" "CRCW0402100KFKEE"
+			(at 203.2 102.87 0)
+			(effects
+				(font
+					(size 1.27 1.27)
+				)
+				(hide yes)
+			)
+		)
 		(pin "2"
 		)
@@
 			)
 		)
+		(property "Part Number" "GRM155R61A106ME11D"
+			(at 164.846 44.45 0)
+			(effects
+				(font
+					(size 1.27 1.27)
+				)
+				(hide yes)
+			)
+		)
 		(pin "2"
 		)
@@
 			)
 		)
+		(property "Alternative PN" "RCC0402200KFKED"
+			(at 236.22 97.79 0)
+			(effects
+				(font
+					(size 1.27 1.27)
+				)
+				(hide yes)
+			)
+		)
+		(property "Part Number" "CRCW0402200KFKEDHP"
+			(at 236.22 97.79 0)
+			(effects
+				(font
+					(size 1.27 1.27)
+				)
+				(hide yes)
+			)
+		)
 		(pin "2"
 		)
@@
 			)
 		)
+		(property "Part Number" "CRCW0402100KFKEE"
+			(at 215.9 118.11 0)
+			(effects
+				(font
+					(size 1.27 1.27)
+				)
+				(hide yes)
+			)
+		)
 		(pin "2"
 		)
@@
 			)
 		)
+		(property "Alternative PN" "RCC0402200KFKED"
+			(at 243.84 97.79 0)
+			(effects
+				(font
+					(size 1.27 1.27)
+				)
+				(hide yes)
+			)
+		)
+		(property "Part Number" "CRCW0402200KFKEDHP"
+			(at 243.84 97.79 0)
+			(effects
+				(font
+					(size 1.27 1.27)
+				)
+				(hide yes)
+			)
+		)
 		(pin "2"
 		)
@@
 			)
 		)
+		(property "Part Number" "GRM1555C2A391JE01D"
+			(at 113.03 104.14 0)
+			(effects
+				(font
+					(size 1.27 1.27)
+				)
+				(hide yes)
+			)
+		)
 		(pin "2"
 		)
@@
 			)
 		)
+		(property "Part Number" "CRCW04020000Z0EDC"
+			(at 205.74 86.36 0)
+			(effects
+				(font
+					(size 1.27 1.27)
+				)
+				(hide yes)
+			)
+		)
 		(pin "2"
 		)
@@
 			)
 		)
+		(property "Part Number" "C3216X5R1E476M160AC"
+			(at 149.606 43.18 0)
+			(effects
+				(font
+					(size 1.27 1.27)
+				)
+				(hide yes)
+			)
+		)
 		(pin "2"
 		)
@@
 		(unit 1)
 		(exclude_from_sim no)
-		(in_bom yes)
+		(in_bom no)
 		(on_board yes)
 		(dnp no)
@@
 			)
 		)
+		(property "Part Number" "GRM155R61A106ME11D"
+			(at 180.594 44.45 0)
+			(effects
+				(font
+					(size 1.27 1.27)
+				)
+				(hide yes)
+			)
+		)
 		(pin "2"
 		)
@@
 			)
 		)
+		(property "Part Number" "CRCW0402100KFKEE"
+			(at 213.36 86.36 0)
+			(effects
+				(font
+					(size 1.27 1.27)
+				)
+				(hide yes)
+			)
+		)
 		(pin "2"
 		)
@@
 			)
 		)
+		(property "Part Number" "CRCW0402100KFKEE"
+			(at 210.82 118.11 0)
+			(effects
+				(font
+					(size 1.27 1.27)
+				)
+				(hide yes)
+			)
+		)
 		(pin "2"
 		)
@@
 			)
 		)
+		(property "Part Number" "GRM188R61E475KE11D"
+			(at 135.89 44.196 0)
+			(effects
+				(font
+					(size 1.27 1.27)
+				)
+				(hide yes)
+			)
+		)
 		(pin "2"
 		)
@@
 			)
 		)
+		(property "Part Number" "CRCW0402100KFKEE"
+			(at 130.81 81.28 0)
+			(effects
+				(font
+					(size 1.27 1.27)
+				)
+				(hide yes)
+			)
+		)
 		(pin "2"
 		)
@@
 			)
 		)
+		(property "Part Number" "TPD4E05U06DQAR"
+			(at 88.9 118.11 0)
+			(effects
+				(font
+					(size 1.27 1.27)
+				)
+				(hide yes)
+			)
+		)
 		(pin "7"
 		)
@@
 		)
 		(property "Description" "Resistor"
+			(at 236.22 113.03 0)
+			(effects
+				(font
+					(size 1.27 1.27)
+				)
+				(hide yes)
+			)
+		)
+		(property "Part Number" "CRCW040210K0FKEDC"
 			(at 236.22 113.03 0)
 			(effects
@@
 				(hide yes)
 			)
+		)
+		(property "Part Number" "TPS25730DREFR"
+			(at 191.77 80.01 0)
+			(effects
+				(font
+					(size 1.27 1.27)
+				)
+				(hide yes)
+			)

Commit message: sch update
Parts:
- R61: value 200k -> 100k
- R7: value 24k -> 10k
Other:
- moved on the sheet: C10, C11, C4, C6, C7, C8, C9, D1, D2, IC8, J7, R45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
