File: PCK-Controller/Controller board/Controller_board/Controller_board.kicad_sch (KiCad schematic)
At the start: 2 parts, among them SW1 SW_Push, U1 EC10E1260507

Commit message: Dimensions draft
Parts:
- removed SW1: SW_Push, SamacSys_Parts.pretty:EVQP0E07K, symbol Switch:SW_Push
- removed U1: EC10E1260507, EC10E1260507, symbol SamacSys_Parts:EC10E1260507
- added H1, H10, H11, H2, H3, H4, H5, H6, H7, H8, H9: MountingHole_Pad, MountingHole:MountingHole_3.2mm_M3_DIN965_Pad, symbol Mechanical:MountingHole_Pad
Other:
- added sheet MCU (MCU.kicad_sch)
- added sheet Power (Power.kicad_sch)

Commit message: .
Other:
- sheet MCU ports: added STM_RX, STM_TX; removed none
- sheet Power ports: added BATT_CE, BATT_ST2, BAT_ST1, CTR_RX, CTR_TX, DN, DP, IN1_SEL, PWR_EN; removed none
Changed lines of the file:
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@@
 	(generator_version "9.0")
 	(paper "A3")
+	(wire
+		(pts
+			(xy 191.77 132.08) (xy 251.46 132.08)
+		)
+		(stroke
+			(width 0)
+			(type default)
+		)
+	)
+	(wire
+		(pts
+			(xy 191.77 129.54) (xy 251.46 129.54)
+		)
+		(stroke
+			(width 0)
+			(type default)
+		)
+	)
 	(symbol
 		(lib_id "Mechanical:MountingHole_Pad")
@@
 	)
 	(sheet
-		(at 227.33 104.14)
-		(size 65.532 34.29)
+		(at 251.46 86.868)
+		(size 64.77 71.12)
 		(exclude_from_sim no)
 		(in_bom yes)
@@
 		)
 		(property "Sheetname" "Power"
-			(at 227.33 103.4284 0)
+			(at 251.46 86.1564 0)
 			(effects
 				(font
@@
 		)
 		(property "Sheetfile" "Power.kicad_sch"
-			(at 227.33 139.0146 0)
+			(at 251.46 158.5726 0)
 			(effects
 				(font
@@
 				)
 				(justify left top)
+			)
+		)
+		(pin "BATT_CE" input
+			(at 251.46 114.3 180)
+			(effects
+				(font
+					(size 1.27 1.27)
+				)
+				(justify left)
+			)
+		)
+		(pin "BATT_ST2" output
+			(at 251.46 119.38 180)
+			(effects
+				(font
+					(size 1.27 1.27)
+				)
+				(justify left)
+			)
+		)
+		(pin "BAT_ST1" output
+			(at 251.46 121.92 180)
+			(effects
+				(font
+					(size 1.27 1.27)
+				)
+				(justify left)
+			)
+		)
+		(pin "CTR_RX" output
+			(at 251.46 129.54 180)
+			(effects
+				(font
+					(size 1.27 1.27)
+				)
+				(justify left)
+			)
+		)
+		(pin "CTR_TX" input
+			(at 251.46 132.08 180)
+			(effects
+				(font
+					(size 1.27 1.27)
+				)
+				(justify left)
+			)
+		)
+		(pin "DN" bidirectional
+			(at 251.46 138.43 180)
+			(effects
+				(font
+					(size 1.27 1.27)
+				)
+				(justify left)
+			)
+		)
+		(pin "DP" bidirectional
+			(at 251.46 140.97 180)
+			(effects
+				(font
+					(size 1.27 1.27)
+				)
+				(justify left)
+			)
+		)
+		(pin "IN1_SEL" output
+			(at 251.46 109.22 180)
+			(effects
+				(font
+					(size 1.27 1.27)
+				)
+				(justify left)
+			)
+		)
+		(pin "PWR_EN" input
+			(at 251.46 105.41 180)
+			(effects
+				(font
+					(size 1.27 1.27)
+				)
+				(justify left)
 			)
 		)
@@
 	(sheet
 		(at 114.808 105.156)
-		(size 77.47 33.274)
+		(size 76.962 33.274)
 		(exclude_from_sim no)
 		(in_bom yes)
@@
 			)
 		)
+		(pin "STM_RX" input
+			(at 191.77 129.54 0)
+			(effects
+				(font
+					(size 1.27 1.27)
+				)
+				(justify right)
+			)
+		)
+		(pin "STM_TX" output
+			(at 191.77 132.08 0)
+			(effects
+				(font
+					(size 1.27 1.27)
+				)
+				(justify right)
+			)
+		)
